Commit message: Added imu

File: urdf/zed_descr.urdf.xacro (robot description, xacro)
@@ -112,4 +112,10 @@
         </joint>
         <link name="$(arg camera_name)_temp_right_link" />
+        <joint name="$(arg camera_name)_imu_joint" type="fixed">
+            <origin xyz="0 0.0093 0" rpy="0 0 0"/>
+            <parent link="$(arg camera_name)_mag_link"/>
+            <child link="$(arg camera_name)_imu_link"/>
+        </joint>
+        <link name="$(arg camera_name)_imu_link"/>
     </xacro:if>
 </robot>
